File: SynthesizerFinal/SynthesizerFinal.kicad_sch (KiCad schematic)
At the start: 274 parts, among them J101 Filter-Send, J102 Filter-Return, J103 Ausgang, J201 Filter-Send, J202 Filter-Return, J203 Ausgang, J301 Filter-Send, J302 Filter-Return, J303 Ausgang, J601 Filter-In, J602 Filter-Out, J701 Filter-In, J702 Filter-Out, J990 Netzteil +/-12V, Q101 BC547, Q201 BC547, Q301 BC547, Q801 BC547, SW101 Wellenform, SW102 weich/hart, SW103 Distortion ein/aus, SW104 Solo-Filter ein/aus, SW201 Wellenform, SW202 weich/hart, SW203 Distortion ein/aus, SW204 Solo-Filter ein/aus, SW301 Wellenform, SW302 weich/hart, SW303 Distortion ein/aus, SW304 Solo-Filter ein/aus, SW401 Filterwahl Ebene A, SW402 Filterwahl Ebene B, SW501 Filterwahl Ebene A, SW502 Filterwahl Ebene B, SW601 Filterwahl Ebene A, SW602 Filterwahl Ebene B, SW701 Filterwahl Ebene A, SW702 Filterwahl Ebene B, U101 LM324, U102 74LVC2G17, U103 OPA4196, U104 OPA1662, U201 LM324, U202 74LVC2G17, U203 OPA4196, U204 OPA1662, U301 LM324, U302 74LVC2G17, U303 OPA4196, U304 OPA1662, U401 ADA4625-2, U501 ADA4625-2, U601 ADA4625-2, U701 ADA4625-2, U901 LM386, U990 78L05

Commit message: 2/3 PCB Designs done, still WIP
Parts:
- removed C405, C505, C605, C705: 680nF, symbol Device:C
- removed C902: 10uF, symbol Device:C_Polarized_US
- removed L401, L403, L501, L503, L601, L603, L701, L703: 33mH, symbol Device:L
- removed L402, L502, L602, L702: 68mH, symbol Device:L
- removed LS901: Speaker 8R, symbol Device:Speaker
- removed SW402, SW502, SW602, SW702: Filterwahl Ebene B, symbol Switch:SW_Rotary_1x5_MP
- removed unit 2 of U401
- removed unit 1 of U401
- removed unit 1 of U501
- removed unit 2 of U501
- removed unit 2 of U601
- removed unit 1 of U601
- removed unit 1 of U701
- removed unit 2 of U701
- added C105, C106, C107, C108, C109, C110, C111, C205, C206, C207, C208, C209, C210, C211, C305, C306, C307, C308, C309, C310, C311, C907: 100nF, Capacitor_THT:C_Disc_D5.0mm_W2.5mm_P5.00mm, symbol Device:C
- added C112, C113, C212, C213, C312, C313, C405, C406, C505, C506, C605, C606, C705, C706: 10uF/25V, Capacitor_THT:CP_Radial_D5.0mm_P2.50mm, symbol Device:C_Polarized_US
- added C906: 100uF/25V, Capacitor_THT:CP_Radial_D6.3mm_P2.50mm, symbol Device:C_Polarized_US
- added D907, D908: 1N5819, Diode_THT:D_DO-41_SOD81_P10.16mm_Horizontal, symbol Diode:1N5819
- added F901, F902: T500mA, Fuse:Fuseholder_Clip-5x20mm_Littelfuse_111_Inline_P20.00x5.00mm_D1.05mm_Horizontal, symbol Device:Fuse
- added J110, J210, J310: Versorgung ein, Connector_JST:JST_XH_B4B-XH-A_1x04_P2.50mm_Vertical, symbol Connector_Generic:Conn_01x04
- added J111, J211, J311: Versorgung weiter, Connector_JST:JST_XH_B4B-XH-A_1x04_P2.50mm_Vertical, symbol Connector_Generic:Conn_01x04
- added J112, J212, J312: Panel Potis, Connector_JST:JST_XH_B11B-XH-A_1x11_P2.50mm_Vertical, symbol Connector_Generic:Conn_01x11
- added J113, J213, J313: Panel Schalter, Connector_JST:JST_XH_B14B-XH-A_1x14_P2.50mm_Vertical, symbol Connector_Generic:Conn_01x14
- added J114, J214, J314: Panel Buchsen, Connector_JST:JST_XH_B6B-XH-A_1x06_P2.50mm_Vertical, symbol Connector_Generic:Conn_01x06
- added J115, J215, J315: Audio aus -> Mixer, Connector_JST:JST_XH_B2B-XH-A_1x02_P2.50mm_Vertical, symbol Connector_Generic:Conn_01x02
- added J410, J510, J610, J710: Versorgung ein, Connector_JST:JST_XH_B3B-XH-A_1x03_P2.50mm_Vertical, symbol Connector_Generic:Conn_01x03
- added J411, J511, J611, J711: Versorgung weiter, Connector_JST:JST_XH_B3B-XH-A_1x03_P2.50mm_Vertical, symbol Connector_Generic:Conn_01x03
- added J412, J512, J612, J712: Panel Poti + Wahlschalter, Connector_JST:JST_XH_B12B-XH-A_1x12_P2.50mm_Vertical, symbol Connector_Generic:Conn_01x12
- added J413, J513, J613, J713: Audio ein, Connector_JST:JST_XH_B2B-XH-A_1x02_P2.50mm_Vertical, symbol Connector_Generic:Conn_01x02
- added J414, J514, J614, J714: Audio aus, Connector_JST:JST_XH_B2B-XH-A_1x02_P2.50mm_Vertical, symbol Connector_Generic:Conn_01x02
- added J810: Versorgung -> Oszillatoren, Connector_JST:JST_XH_B4B-XH-A_1x04_P2.50mm_Vertical, symbol Connector_Generic:Conn_01x04
- added J811: Versorgung -> Filter, Connector_JST:JST_XH_B3B-XH-A_1x03_P2.50mm_Vertical, symbol Connector_Generic:Conn_01x03
- added J812: Panel Potis, Connector_JST:JST_XH_B12B-XH-A_1x12_P2.50mm_Vertical, symbol Connector_Generic:Conn_01x12
- added J813: OSC 1 ein, Connector_JST:JST_XH_B2B-XH-A_1x02_P2.50mm_Vertical, symbol Connector_Generic:Conn_01x02
- added J814: OSC 2 ein, Connector_JST:JST_XH_B2B-XH-A_1x02_P2.50mm_Vertical, symbol Connector_Generic:Conn_01x02
- added J815: OSC 3 ein, Connector_JST:JST_XH_B2B-XH-A_1x02_P2.50mm_Vertical, symbol Connector_Generic:Conn_01x02
- added J816: -> Filter A, Connector_JST:JST_XH_B2B-XH-A_1x02_P2.50mm_Vertical, symbol Connector_Generic:Conn_01x02
- added J817: Filter B ->, Connector_JST:JST_XH_B2B-XH-A_1x02_P2.50mm_Vertical, symbol Connector_Generic:Conn_01x02
- added J904: Lautsprecher 8R, Connector_JST:JST_XH_B2B-XH-A_1x02_P2.50mm_Vertical, symbol Connector_Generic:Conn_01x02
- added R404, R406, R408, R409, R410, R504, R506, R508, R509, R510, R604, R606, R608, R609, R610, R704, R706, R708, R709, R710: 10k, Resistor_THT:R_Axial_DIN0207_L6.3mm_D2.5mm_P7.62mm_Horizontal, symbol Device:R_US
- added R407, R507, R607, R707: 6.8k, Resistor_THT:R_Axial_DIN0207_L6.3mm_D2.5mm_P7.62mm_Horizontal, symbol Device:R_US
- added R902: 68k, Resistor_THT:R_Axial_DIN0207_L6.3mm_D2.5mm_P7.62mm_Horizontal, symbol Device:R_US
- added unit 1 of U401
- added unit 2 of U401
- added unit 3 of U401
- added unit 4 of U401
- added unit 1 of U501
- added unit 2 of U501
- added unit 3 of U501
- added unit 4 of U501
- added unit 1 of U601
- added unit 2 of U601
- added unit 3 of U601
- added unit 4 of U601
- added unit 1 of U701
- added unit 2 of U701
- added unit 3 of U701
- added unit 4 of U701
- C101, C201, C301: value 33nF -> 47nF; footprint (none) -> Capacitor_THT:C_Rect_L7.0mm_W2.5mm_P5.00mm
- C102, C202, C302, C401, C402, C501, C502, C601, C602, C701, C702, C905, C941: footprint (none) -> Capacitor_THT:C_Rect_L7.0mm_W2.5mm_P5.00mm
- C103, C104, C203, C204, C303, C304, C801, C802, C803: footprint (none) -> Capacitor_THT:C_Rect_L7.0mm_W4.5mm_P5.00mm
- C403, C503, C603, C703, C921, C922, C942: footprint (none) -> Capacitor_THT:C_Disc_D5.0mm_W2.5mm_P5.00mm
- C404, C504, C604, C704: value 220nF -> 100nF; footprint (none) -> Capacitor_THT:C_Disc_D5.0mm_W2.5mm_P5.00mm
- C804, C903: value 10uF -> 10uF/16V; footprint (none) -> Capacitor_THT:CP_Radial_D5.0mm_P2.50mm
- C805: value 470uF -> 470uF/16V; footprint (none) -> Capacitor_THT:CP_Radial_D10.0mm_P5.00mm
- C806: value 47uF -> 47uF/25V; footprint (none) -> Capacitor_THT:CP_Radial_D6.3mm_P2.50mm
- C901: value 10uF -> 10uF/25V bipolar; footprint (none) -> Capacitor_THT:CP_Radial_D5.0mm_P2.50mm; symbol Device:C_Polarized_US -> Device:C
- C904: value 220uF -> 470uF/25V; footprint (none) -> Capacitor_THT:CP_Radial_D10.0mm_P5.00mm
- C931, C932: value 100uF -> 100uF/25V; footprint (none) -> Capacitor_THT:CP_Radial_D6.3mm_P2.50mm
- D101, D102, D103, D104, D105, D106, D201, D202, D203, D204, D205, D206, D301, D302, D303, D304, D305, D306: footprint (none) -> Diode_THT:D_DO-35_SOD27_P7.62mm_Horizontal; symbol Diode:1N4148WT -> Diode:1N4148
- J990: footprint (none) -> Connector_JST:JST_XH_B3B-XH-A_1x03_P2.50mm_Vertical
- Q101, Q201, Q301, Q801, U990: footprint (none) -> Package_TO_SOT_THT:TO-92_Inline_Wide
- R101, R102, R103, R104, R106, R107, R108, R109, R110, R111, R113, R114, R116, R117, R118, R119, R120, R121, R122, R123, R125, R127, R201, R202, R203, R204, R206, R207, R208, R209, R210, R211, R213, R214, R216, R217, R218, R219, R220, R221, R222, R223, R225, R227, R301, R302, R303, R304, R306, R307, R308, R309, R310, R311, R313, R314, R316, R317, R318, R319, R320, R321, R322, R323, R325, R327: footprint (none) -> Resistor_THT:R_Axial_DIN0207_L6.3mm_D2.5mm_P2.54mm_Vertical
- R105, R205, R305: value 18k -> 16k; footprint (none) -> Resistor_THT:R_Axial_DIN0207_L6.3mm_D2.5mm_P2.54mm_Vertical
- R112, R212, R312: value 47k -> 82k; footprint (none) -> Resistor_THT:R_Axial_DIN0207_L6.3mm_D2.5mm_P2.54mm_Vertical
- R115, R215, R315: value 100k -> 330k; footprint (none) -> Resistor_THT:R_Axial_DIN0207_L6.3mm_D2.5mm_P2.54mm_Vertical
- R124, R224, R324: value 68k -> 110k; footprint (none) -> Resistor_THT:R_Axial_DIN0207_L6.3mm_D2.5mm_P2.54mm_Vertical
- R126, R226, R326: value 22k -> 20k; footprint (none) -> Resistor_THT:R_Axial_DIN0207_L6.3mm_D2.5mm_P2.54mm_Vertical
- R401, R402, R405, R501, R502, R505, R601, R602, R605, R701, R702, R705, R804, R805, R901: footprint (none) -> Resistor_THT:R_Axial_DIN0207_L6.3mm_D2.5mm_P7.62mm_Horizontal
- R403, R503, R603, R703: value 600 -> 6.8k; footprint (none) -> Resistor_THT:R_Axial_DIN0207_L6.3mm_D2.5mm_P7.62mm_Horizontal
- R801, R802, R803: value 22k -> 100k; footprint (none) -> Resistor_THT:R_Axial_DIN0207_L6.3mm_D2.5mm_P7.62mm_Horizontal
- R806: value 330 -> 470; footprint (none) -> Resistor_THT:R_Axial_DIN0207_L6.3mm_D2.5mm_P7.62mm_Horizontal
- R807: value 10 -> 100; footprint (none) -> Resistor_THT:R_Axial_DIN0207_L6.3mm_D2.5mm_P7.62mm_Horizontal
- R808: value 90 -> 1; footprint (none) -> Resistor_THT:R_Axial_DIN0207_L6.3mm_D2.5mm_P7.62mm_Horizontal
- R809: value 1k -> 100k; footprint (none) -> Resistor_THT:R_Axial_DIN0207_L6.3mm_D2.5mm_P7.62mm_Horizontal
- RV103, RV203, RV303, RV401, RV402, RV501, RV502, RV601, RV602, RV701, RV702: value 100k -> 100k lin
- RV104, RV204, RV304: value 100k -> 100k log
- RV403, RV503, RV603, RV703: value 47k -> 47k lin
- RV801, RV802, RV803, RV901: value 10k -> 10k log
- SW401, SW501, SW601, SW701: value Filterwahl Ebene A -> Filterwahl
- U101, U201, U301: value LM324 -> TL074; footprint (none) -> Package_DIP:DIP-14_W7.62mm_Socket; symbol Amplifier_Operational:LM324 -> Amplifier_Operational:TL074
- U102, U202, U302: footprint (none) -> Package_TO_SOT_SMD:SOT-363_SC-70-6
- U103, U203, U303: footprint (none) -> Package_SO:SOIC-14_3.9x8.7mm_P1.27mm; symbol Amplifier_Operational:OPA4196xPW -> Amplifier_Operational:OPA4196xD
- U103, U203, U303: value OPA4196xPW -> OPA4196; footprint (none) -> Package_SO:SOIC-14_3.9x8.7mm_P1.27mm; symbol Amplifier_Operational:OPA4196xPW -> Amplifier_Operational:OPA4196xD
- U104, U204, U304: footprint (none) -> Package_SO:SOIC-8_3.9x4.9mm_P1.27mm
- U104, U204, U304: value OPA1662D -> OPA1662; footprint (none) -> Package_SO:SOIC-8_3.9x4.9mm_P1.27mm
- U401, U501, U601, U701: value ADA4625-2ARDZ -> OPA4196; footprint (none) -> Package_SO:SOIC-14_3.9x8.7mm_P1.27mm; symbol Amplifier_Operational:ADA4625-2ARDZ -> Amplifier_Operational:OPA4196xD
- U901: footprint (none) -> Package_DIP:DIP-8_W7.62mm_Socket
Connections:
- net +12V: now also C403.1, C503.1, C603.1, C703.1, U401.4 (V+), U501.4 (V+), U601.4 (V+), U701.4 (V+), C105.1, C108.1, C110.1, C112.1, C205.1, C208.1, C210.1, C212.1, C305.1, C308.1, C310.1, C312.1, C405.1, C505.1, C605.1, C705.1, C906.1, C907.1, D907.1 (K), J110.1 (Pin_1), J111.1 (Pin_1), J210.1 (Pin_1), J211.1 (Pin_1), J310.1 (Pin_1), J311.1 (Pin_1), J410.1 (Pin_1), J411.1 (Pin_1), J510.1 (Pin_1), J511.1 (Pin_1), J610.1 (Pin_1), J611.1 (Pin_1), J710.1 (Pin_1), J711.1 (Pin_1), J810.1 (Pin_1), J811.1 (Pin_1); no longer J990.1 (Pin_1), U401.8 (V+), U501.8 (V+), U601.8 (V+), U701.8 (V+)
- net +5V: now also C107.1, C207.1, C307.1, J110.4 (Pin_4), J111.4 (Pin_4), J112.5 (Pin_5), J210.4 (Pin_4), J211.4 (Pin_4), J212.5 (Pin_5), J310.4 (Pin_4), J311.4 (Pin_4), J312.5 (Pin_5), J810.4 (Pin_4)
- net -12V: now also C404.2, C504.2, C604.2, C704.2, U401.11 (V-), U501.11 (V-), U601.11 (V-), U701.11 (V-), C106.2, C109.2, C111.2, C113.2, C206.2, C209.2, C211.2, C213.2, C306.2, C309.2, C311.2, C313.2, C406.2, C506.2, C606.2, C706.2, D908.2 (A), J110.3 (Pin_3), J111.3 (Pin_3), J210.3 (Pin_3), J211.3 (Pin_3), J310.3 (Pin_3), J311.3 (Pin_3), J410.3 (Pin_3), J411.3 (Pin_3), J510.3 (Pin_3), J511.3 (Pin_3), J610.3 (Pin_3), J611.3 (Pin_3), J710.3 (Pin_3), J711.3 (Pin_3), J810.3 (Pin_3), J811.3 (Pin_3); no longer J990.3 (Pin_3), U401.4 (V-), U501.4 (V-), U601.4 (V-), U701.4 (V-)
- net FILT_A_OUT: now also SW401.6, SW501.5, J412.12 (Pin_12), J414.1 (Pin_1), J512.11 (Pin_11), J513.1 (Pin_1), R504.1; no longer RV403.2
- net FILT_B_OUT: now also SW501.6, J512.12 (Pin_12), J514.1 (Pin_1), J817.1 (Pin_1); no longer RV503.2
- net GNDREF: now also C404.1, C504.1, C604.1, C704.1, C105.2, C106.1, C107.2, C108.2, C109.1, C110.2, C111.1, C112.2, C113.1, C205.2, C206.1, C207.2, C208.2, C209.1, C210.2, C211.1, C212.2, C213.1, C305.2, C306.1, C307.2, C308.2, C309.1, C310.2, C311.1, C312.2, C313.1, C405.2, C406.1, C505.2, C506.1, C605.2, C606.1, C705.2, C706.1, C906.2, C907.2, J110.2 (Pin_2), J111.2 (Pin_2), J112.8 (Pin_8), J114.2 (Pin_2), J114.4 (Pin_4), J114.6 (Pin_6), J115.2 (Pin_2), J210.2 (Pin_2), J211.2 (Pin_2), J212.8 (Pin_8), J214.2 (Pin_2), J214.4 (Pin_4), J214.6 (Pin_6), J215.2 (Pin_2), J310.2 (Pin_2), J311.2 (Pin_2), J312.8 (Pin_8), J314.2 (Pin_2), J314.4 (Pin_4), J314.6 (Pin_6), J315.2 (Pin_2), J410.2 (Pin_2), J411.2 (Pin_2), J413.2 (Pin_2), J414.2 (Pin_2), J510.2 (Pin_2), J511.2 (Pin_2), J513.2 (Pin_2), J514.2 (Pin_2), J610.2 (Pin_2), J611.2 (Pin_2), J613.2 (Pin_2), J614.2 (Pin_2), J710.2 (Pin_2), J711.2 (Pin_2), J713.2 (Pin_2), J714.2 (Pin_2), J810.2 (Pin_2), J811.2 (Pin_2), J812.12 (Pin_12), J812.3 (Pin_3), J812.6 (Pin_6), J812.9 (Pin_9), J813.2 (Pin_2), J814.2 (Pin_2), J815.2 (Pin_2), J816.2 (Pin_2), J817.2 (Pin_2), J904.2 (Pin_2), R407.1, R507.1, R607.1, R707.1, U401.10 (+), U401.12 (+), U401.5 (+), U501.10 (+), U501.12 (+), U501.5 (+), U601.10 (+), U601.12 (+), U601.5 (+), U701.10 (+), U701.12 (+), U701.5 (+); no longer C401.2, C501.2, C601.2, C701.2, R402.2, R403.2, R405.2, R502.2, R503.2, R505.2, R602.2, R603.2, R605.2, R702.2, R703.2, R705.2
- net MIX_OUT: now also SW401.5, J412.11 (Pin_11), J413.1 (Pin_1), J816.1 (Pin_1), R404.1
- net OSC1_DIST: now also J113.11 (Pin_11), J113.2 (Pin_2)
- net OSC1_OUT: now also J114.5 (Pin_5), J115.1 (Pin_1), J813.1 (Pin_1)
- net OSC1_SAW: now also J113.8 (Pin_8)
- net OSC1_SIG: now also J113.12 (Pin_12), J114.3 (Pin_3)
- net OSC1_SINE: now also J113.13 (Pin_13)
- net OSC1_SQ: now also J113.9 (Pin_9)
- net OSC1_TRI: now also J113.10 (Pin_10)
- net OSC1_WAVE: now also J113.4 (Pin_4); no longer RV104.1
- net OSC2_DIST: now also J213.11 (Pin_11), J213.2 (Pin_2)
- net OSC2_OUT: now also J214.5 (Pin_5), J215.1 (Pin_1), J814.1 (Pin_1)
- net OSC2_SAW: now also J213.8 (Pin_8)
- net OSC2_SIG: now also J213.12 (Pin_12), J214.3 (Pin_3)
- net OSC2_SINE: now also J213.13 (Pin_13)
- net OSC2_SQ: now also J213.9 (Pin_9)
- net OSC2_TRI: now also J213.10 (Pin_10)
- net OSC2_WAVE: now also J213.4 (Pin_4); no longer RV204.1
- net OSC3_DIST: now also J313.11 (Pin_11), J313.2 (Pin_2)
- net OSC3_OUT: now also J314.5 (Pin_5), J315.1 (Pin_1), J815.1 (Pin_1)
- net OSC3_SAW: now also J313.8 (Pin_8)
- net OSC3_SIG: now also J313.12 (Pin_12), J314.3 (Pin_3)
- net OSC3_SINE: now also J313.13 (Pin_13)
- net OSC3_SQ: now also J313.9 (Pin_9)
- net OSC3_TRI: now also J313.10 (Pin_10)
- net OSC3_WAVE: now also J313.4 (Pin_4); no longer RV304.1
- net F6_LP: now reaches SW601.1
- net F6_LP: now also C602.2, R605.1, J612.7 (Pin_7), R609.1, U601.8; no longer R601.1
- net at R601.2: now also C601.1, U601.6 (-); no longer RV601.1
- net O2_WSEL: now reaches C203.1, SW201.5
- net O2_WSEL: now also J213.3 (Pin_3)
- net O3_DRIVE: now reaches RV303.2, SW302.3 (A), U303.1
- net O3_DRIVE: now also R316.1, J312.4 (Pin_4), J313.7 (Pin_7); no longer D303.2 (A), D304.1 (K)
- net O3_AINV: now reaches D303.1 (K), D304.2 (A), R314.2, RV303.1, U303.2 (-)
- net O3_AINV: now also SW302.1 (C), J312.3 (Pin_3), J313.5 (Pin_5)
- net O3_LVL_A: now reaches R320.2, RV305.1, U304.1
- net O3_LVL_A: now also J312.10 (Pin_10)
- net O3_LVL_W: now reaches RV305.2, U304.5 (+)
- net O3_LVL_W: now also J312.11 (Pin_11)
- net O3_FGF_A: now reaches R306.2, RV302.1
- net O3_FGF_A: now also J312.7 (Pin_7)
- net O3_PITCH: now reaches R301.1, RV301.2
- net O3_PITCH: now also J312.6 (Pin_6)
- net O1_AINV: now reaches D103.1 (K), D104.2 (A), R114.2, RV103.1, U103.2 (-)
- net O1_AINV: now also SW102.1 (C), J112.3 (Pin_3), J113.5 (Pin_5)
- net O1_DRIVE: now reaches RV103.2, SW102.3 (A), U103.1
- net O1_DRIVE: now also R116.1, J112.4 (Pin_4), J113.7 (Pin_7); no longer D103.2 (A), D104.1 (K)
- net F6_NOTCH: now reaches SW601.4
- net F6_NOTCH: now also J612.10 (Pin_10), R610.2, U601.14
- net F6_RESW: now reaches R603.1
- net F6_RESW: now also RV603.2, J612.6 (Pin_6)
- net F4_NOTCH: now reaches SW401.4
- net F4_NOTCH: now also J412.10 (Pin_10), R410.2, U401.14
- net F4_RESW: now reaches R403.1
- net F4_RESW: now also RV403.2, J412.6 (Pin_6)
- net O3_CLIP: now reaches D305.1 (K), D306.2 (A), R316.2
- net O3_CLIP: now also RV304.1, J312.1 (Pin_1); no longer SW302.1 (C)
- net O2_AINV: now reaches D203.1 (K), D204.2 (A), R214.2, RV203.1, U203.2 (-)
- net O2_AINV: now also SW202.1 (C), J212.3 (Pin_3), J213.5 (Pin_5)
- net O2_DRIVE: now reaches RV203.2, SW202.3 (A), U203.1
- net O2_DRIVE: now also R216.1, J212.4 (Pin_4), J213.7 (Pin_7); no longer D203.2 (A), D204.1 (K)
- net O1_WSEL: now reaches C103.1, SW101.5
- net O1_WSEL: now also J113.3 (Pin_3)
- net F5_BP: now reaches RV503.1
- net F5_BP: now also C501.2, RV502.1, SW501.3, J512.3 (Pin_3), J512.5 (Pin_5), J512.9 (Pin_9), U501.7; no longer R505.1
- net O2_MKUP_A: now reaches R215.1, RV204.2, U203.6 (-)
- net O2_MKUP_A: now also J212.2 (Pin_2)
- net O2_MKUP: now reaches R215.2, U203.7
- net O2_MKUP: now also SW203.1 (C), J213.6 (Pin_6); no longer R216.1
- net F6_BP: now reaches RV603.1
- net F6_BP: now also C601.2, RV602.1, SW601.3, J612.3 (Pin_3), J612.5 (Pin_5), J612.9 (Pin_9), U601.7; no longer R605.1
- net F6_OUT: now reaches J602.T
- net F6_OUT: now also SW601.6, J612.12 (Pin_12), J614.1 (Pin_1); no longer RV603.2
- net F7_BP: now reaches RV703.1
- net F7_BP: now also C701.2, RV702.1, SW701.3, J712.3 (Pin_3), J712.5 (Pin_5), J712.9 (Pin_9), U701.7; no longer R705.1
- net F7_OUT: now reaches J702.T
- net F7_OUT: now also SW701.6, J712.12 (Pin_12), J714.1 (Pin_1); no longer RV703.2
- net F6_T2W: now reaches R602.1, RV602.2
- net F6_T2W: now also J612.4 (Pin_4)
- net at C602.1: now also R602.2, U601.9 (-); no longer SW601.2
- net O1_SEND: now reaches J101.T, SW104.1 (C)
- net O1_SEND: now also J113.14 (Pin_14), J114.1 (Pin_1)
- net O2_FGF_A: now reaches R206.2, RV202.1
- net O2_FGF_A: now also J212.7 (Pin_7)
- net at C401.1: now also R401.2, U401.6 (-); no longer RV401.2
- net F7_LP: now reaches SW701.1
- net F7_LP: now also C702.2, R705.1, J712.7 (Pin_7), R709.1, U701.8; no longer R701.1
- net at C702.1: now also R702.2, U701.9 (-); no longer SW701.2
- net F7_NOTCH: now reaches SW701.4
- net F7_NOTCH: now also J712.10 (Pin_10), R710.2, U701.14
- net F7_IN: now reaches SW701.5
- net F7_IN: now also J701.T, J712.11 (Pin_11), J713.1 (Pin_1), R704.1
- net O1_MKUP_A: now reaches R115.1, RV104.2, U103.6 (-)
- net O1_MKUP_A: now also J112.2 (Pin_2)
- net O1_MKUP: now reaches R115.2, U103.7
- net O1_MKUP: now also SW103.1 (C), J113.6 (Pin_6); no longer R116.1
- net M_LVL3_A: now reaches C803.2, RV803.1
- net M_LVL3_A: now also J812.7 (Pin_7)
- net M_LVL3_W: now reaches R803.1, RV803.2
- net M_LVL3_W: now also J812.8 (Pin_8)
- net O3_FGF_B: now reaches C302.1, RV302.2, U301.6 (-)
- net O3_FGF_B: now also J312.9 (Pin_9)
- net O3_MKUP: now reaches SW303.1 (C)
- net O3_MKUP: now also R315.2, U303.7, J313.6 (Pin_6); no longer SW302.2 (B)
- net O2_SOFT: now reaches SW202.2 (B)
- net O2_SOFT: now also D203.2 (A), D204.1 (K), J213.1 (Pin_1); no longer SW203.1 (C)
- net M_LVL1_A: now reaches C801.2, RV801.1
- net M_LVL1_A: now also J812.1 (Pin_1)
- net at R701.2: now also C701.1, U701.6 (-); no longer RV701.1
- net F6_IN: now reaches J601.T
- net F6_IN: now also SW601.5, J612.11 (Pin_11), J613.1 (Pin_1), R604.1
- net F6_T1W: now reaches RV601.2
- net F6_T1W: now also R601.1, J612.2 (Pin_2); no longer C601.1
- net O2_PITCH: now reaches R201.1, RV201.2
- net O2_PITCH: now also J212.6 (Pin_6)
- net F4_HP: now reaches RV401.1
- net F4_HP: now also SW401.2, J412.1 (Pin_1), J412.8 (Pin_8), R406.1, R408.1, U401.1; no longer R401.2
- net M_LVL1_W: now reaches R801.1, RV801.2
- net M_LVL1_W: now also J812.2 (Pin_2)
- net at R801.2, R802.2, R803.2: now also C804.2; no longer C804.1
- net O2_CLIP: now reaches D205.1 (K), D206.2 (A), R216.2
- net O2_CLIP: now also RV204.1, J212.1 (Pin_1); no longer SW202.1 (C)
- net F5_LP: now reaches SW501.1
- net F5_LP: now also C502.2, R505.1, J512.7 (Pin_7), R509.1, U501.8; no longer R501.1
- net at R501.2: now also C501.1, U501.6 (-); no longer RV501.1
- net F7_T1W: now reaches RV701.2
- net F7_T1W: now also R701.1, J712.2 (Pin_2); no longer C701.1
- net F4_BP: now reaches RV402.1
- net F4_BP: now also C401.2, RV403.1, SW401.3, J412.3 (Pin_3), J412.5 (Pin_5), J412.9 (Pin_9), U401.7; no longer C402.2
- net F4_T2W: now reaches R402.1, RV402.2
- net F4_T2W: now also J412.4 (Pin_4)
- net O2_LVL_A: now reaches R220.2, RV205.1, U204.1
- net O2_LVL_A: now also J212.10 (Pin_10)
- net F5_T1W: now reaches RV501.2
- net F5_T1W: now also R501.1, J512.2 (Pin_2); no longer C501.1
- net O3_MKUP_A: now reaches R315.1, RV304.2, U303.6 (-)
- net O3_MKUP_A: now also J312.2 (Pin_2)
- net at Q801.2 (B), R804.2, R805.1: now also C804.1; no longer C804.2
- net O1_FGF_B: now reaches C102.1, RV102.2, U101.6 (-)
- net O1_FGF_B: now also J112.9 (Pin_9)
- net at C502.1: now also R502.2, U501.9 (-); no longer SW501.2
- net F5_NOTCH: now reaches SW501.4
- net F5_NOTCH: now also J512.10 (Pin_10), R510.2, U501.14
- net at C402.1: now also R402.2, U401.9 (-); no longer SW401.2
- net F5_RESW: now reaches R503.1
- net F5_RESW: now also RV503.2, J512.6 (Pin_6)
- net O1_CLIP: now reaches D105.1 (K), D106.2 (A), R116.2
- net O1_CLIP: now also RV104.1, J112.1 (Pin_1); no longer SW102.1 (C)
- net O1_PITCH: now reaches R101.1, RV101.2
- net O1_PITCH: now also J112.6 (Pin_6)
- net F4_LP: now reaches R405.1
- net F4_LP: now also C402.2, SW401.1, J412.7 (Pin_7), R409.1, U401.8; no longer RV403.1
- net O3_SEND: now reaches J301.T, SW304.1 (C)
- net O3_SEND: now also J313.14 (Pin_14), J314.1 (Pin_1)
- net F5_T2W: now reaches R502.1, RV502.2
- net F5_T2W: now also J512.4 (Pin_4)
- net M_LVL2_A: now reaches C802.2, RV802.1
- net M_LVL2_A: now also J812.4 (Pin_4)
- net M_LVL2_W: now reaches R802.1, RV802.2
- net M_LVL2_W: now also J812.5 (Pin_5)
- net F7_RESW: now reaches R703.1
- net F7_RESW: now also RV703.2, J712.6 (Pin_6)
- net O1_LVL_A: now reaches R120.2, RV105.1, U104.1
- net O1_LVL_A: now also J112.10 (Pin_10)
- net O1_LVL_W: now reaches RV105.2, U104.5 (+)
- net O1_LVL_W: now also J112.11 (Pin_11)
- net F7_T2W: now reaches R702.1, RV702.2
- net F7_T2W: now also J712.4 (Pin_4)
- net F4_T1W: now reaches R401.1
- net F4_T1W: now also RV401.2, J412.2 (Pin_2); no longer SW401.1
- net at C901.2: now also R902.1; no longer RV901.1
- net O3_WSEL: now reaches C303.1, SW301.5
- net O3_WSEL: now also J313.3 (Pin_3)
- net O2_FGF_B: now reaches C202.1, RV202.2, U201.6 (-)
- net O2_FGF_B: now also J212.9 (Pin_9)
- net O2_LVL_W: now reaches RV205.2, U204.5 (+)
- net O2_LVL_W: now also J212.11 (Pin_11)
- net O1_FGF_A: now reaches R106.2, RV102.1
- net O1_FGF_A: now also J112.7 (Pin_7)
- net M_VOL_W: now reaches RV901.2, U901.3 (+)
- net M_VOL_W: now also J812.11 (Pin_11)
- net at C904.2: now also J904.1 (Pin_1)
- net O1_SOFT: now reaches SW102.2 (B)
- net O1_SOFT: now also D103.2 (A), D104.1 (K), J113.1 (Pin_1); no longer SW103.1 (C)
- net O2_SEND: now reaches J201.T, SW204.1 (C)
- net O2_SEND: now also J213.14 (Pin_14), J214.1 (Pin_1)
- new net: R404.2, R405.2, R406.2, U401.2 (-)
- new net: R403.2, R407.2, U401.3 (+)
- new net: R408.2, R409.2, R410.1, U401.13 (-)
- new net: R504.2, R505.2, R506.2, U501.2 (-)
- new net: R503.2, R507.2, U501.3 (+)
- new net: R508.2, R509.2, R510.1, U501.13 (-)
- new net: R604.2, R605.2, R606.2, U601.2 (-)
- new net: R603.2, R607.2, U601.3 (+)
- new net: R608.2, R609.2, R610.1, U601.13 (-)
- new net: R704.2, R705.2, R706.2, U701.2 (-)
- new net: R703.2, R707.2, U701.3 (+)
- new net: R708.2, R709.2, R710.1, U701.13 (-)
- new net: D907.2 (A), F901.2
- new net: D908.1 (K), F902.2
- new net F5_HP: J512.1 (Pin_1), J512.8 (Pin_8), R506.1, R508.1, RV501.1, SW501.2, U501.1
- new net F6_HP: J612.1 (Pin_1), J612.8 (Pin_8), R606.1, R608.1, RV601.1, SW601.2, U601.1
- new net F7_HP: J712.1 (Pin_1), J712.8 (Pin_8), R706.1, R708.1, RV701.1, SW701.2, U701.1
- new net M_VOL_A: J812.10 (Pin_10), R902.2, RV901.1
- new net O3_SOFT: D303.2 (A), D304.1 (K), J313.1 (Pin_1), SW302.2 (B)
- new net VIN_N: F902.1, J990.3 (Pin_3)
- new net VIN_P: F901.1, J990.1 (Pin_1)
- no-connect marks 18 -> 12
Other:
- note added: "Entkopplung Filter A / B"
- note added: "Entkopplung Filter C / D"
- note added: "Entkopplung OSC 1"
- note added: "Entkopplung OSC 2"
- note added: "Entkopplung OSC 3"
- note added: "F901/F902 begrenzen den Strom bei einem Kurzschluss. D907/D908 (Schottky) sperren, wenn der Netzstecker verpolt ist: +12 V und -12 V koennen dann nicht vertauscht an die ICs gelangen. Spannungsverlust ca. 0,3 V pro Schiene."
- note added: "FILTER A (Hauptweg 1 von 2) - State-Variable-Filter"
- note added: "FILTER B (Hauptweg 2 von 2) - State-Variable-Filter"
- note added: "FILTER C (Solo-Filter 1) - State-Variable-Filter"
- note added: "FILTER D (Solo-Filter 2) - State-Variable-Filter"
- note added: "Filter A"
- note added: "Filter B"
- note added: "Filter C"
- note added: "Filter D"
- note added: "Mixer / Endstufe"
- note added: "OSC 1"
- note added: "OSC 2"
- note added: "OSC 3"
- note added: "RV901 = Master-Lautstaerke (log). R902 daempft den Filterpegel ab. Pin 1-8 offen -> Verstaerkung 20. R901/C905 = Zobel-Glied. C906/C907 = lokale Abblockung direkt am LM386 (Pin 6). Bei +12 V die Variante LM386N-4 verwenden (Datenblatt pruefen)."
- note added: "VERPOLUNGS- UND UEBERSTROMSCHUTZ"
- note removed: "Bandpass ca. 650 Hz .. 5.5 kHz"
- note removed: "Bandsperre Kerbe bei ca. 1.06 kHz"
- note removed: "Eingangspuffer U401B, Ausgangsverstaerker U401A. RV401/RV402 = gemeinsames Cutoff-Poti (2-fach-Gleichlauf)."
- note removed: "FILTER C (Solo-Filter 1)"
- note removed: "Hochpass 106 Hz .. 10.6 kHz"
- note removed: "RV901 = Master-Lautstaerke. C902 (Pin 1-8) -> Verstaerkung 200. R901/C905 = Zobel-Glied zur Stabilisierung."
- note removed: "Tiefpass 106 Hz .. 10.6 kHz"
- moved on the sheet: C804
